File: rp2040_stamp_round.kicad_pcb (KiCad board)
At the start: 4 copper layers, 60 x 60 mm, 104 parts, among them J1 Conn_01x01, J10 Conn_01x01, J11 Conn_01x01, J12 Conn_01x01, J13 Conn_01x01, J14 Conn_01x01, J15 Conn_01x01, J16 Conn_01x01, J17 Conn_01x01, J18 Conn_01x01, J19 USB_C_Receptacle_USB2.0, J2 Conn_01x01, J20 Conn_Batt, J3 Conn_01x01, J4 Conn_01x01, J5 Conn_01x01, J6 Conn_01x01, J7 Conn_01x01, J8 Conn_01x01, J9 Conn_01x01, SW1 SW_OnOff, SW2 SW_SPST, SW3 SW_SPST, U1 RP2040_Stamp

Commit message: Production rev release
Parts:
- removed kibuzzard-61B7F843 (x2): G***, kibuzzard-61B7F843
- removed kibuzzard-61BA2B2B (x2): G***, kibuzzard-61BA2B2B
- added JP1: Jumper_PWR, Jumper:SolderJumper-2_P1.3mm_Bridged_RoundedPad1.0x1.5mm, B.Cu at (145.2, 68.2)
- added TP1: TP_BOOTSEL, TestPoint:TestPoint_Pad_D2.0mm, B.Cu at (139.7, 74.0)
- added kibuzzard-61DD9534: G***, kibuzzard-61DD9534, F.Cu at (167.1, 109.8)
- added kibuzzard-61DD9534: G***, kibuzzard-61DD9534, B.Cu at (167.1, 109.8)
- added kibuzzard-61DD9594: G***, kibuzzard-61DD9594, F.Cu at (135.1, 96.0)
- added kibuzzard-61DD95B3: G***, kibuzzard-61DD95B3, B.Cu at (170.3, 91.6)
- added kibuzzard-61DD95E6: G***, kibuzzard-61DD95E6, B.Cu at (157.8, 64.8)
- added kibuzzard-61DD95F0: G***, kibuzzard-61DD95F0, B.Cu at (145.2, 64.8)
- added kibuzzard-61E03091: G***, kibuzzard-61E03091, B.Cu at (139.7, 75.9)
- added kibuzzard-61E0313F: G***, kibuzzard-61E0313F, B.Cu at (139.7, 77.4)
- moved kibuzzard-61BA2B21 0.20 mm to (169.0, 91.5)
Connections:
- D17 pad 1: GND -> Net-(D17-K)
- U1 pad 40: unconnected-(U1-Pad40) -> Net-(U1-BOOTSEL)
Routing:
- net Net-(U1-BOOTSEL): track 0.00 -> 7.01 mm
- net Net-(D17-K): track 0.00 -> 5.86 mm, vias 0 -> 1
- net unconnected-(U1-Pad40): track 1.55 -> 0.00 mm
- net GND: track 28.7 -> 29.8 mm, vias 25 -> 24
- net +3V3: track 20.3 -> 20.9 mm
