File: rp2040_stamp_round.kicad_sch (KiCad schematic)
At the start: 46 parts, among them J1 Conn_01x01, J10 Conn_01x01, J11 Conn_01x01, J12 Conn_01x01, J13 Conn_01x01, J14 Conn_01x01, J15 Conn_01x01, J16 Conn_01x01, J17 Conn_01x01, J18 Conn_01x01, J19 USB_C_Receptacle_USB2.0, J2 Conn_01x01, J20 Conn_Batt, J3 Conn_01x01, J4 Conn_01x01, J5 Conn_01x01, J6 Conn_01x01, J7 Conn_01x01, J8 Conn_01x01, J9 Conn_01x01, SW1 SW_OnOff, SW2 SW_SPST, SW3 SW_SPST, U1 RP2040_Stamp

Commit message: Production rev release
Parts:
- added JP1: Jumper_PWR, Jumper:SolderJumper-2_P1.3mm_Bridged_RoundedPad1.0x1.5mm, symbol Jumper:Jumper_2_Bridged
- added TP1: TP_BOOTSEL, TestPoint:TestPoint_Pad_D2.0mm, symbol Connector:TestPoint
- D1, D10, D11, D12, D13, D14, D15, D16, D2, D3, D4, D5, D6, D7, D8, D9: LCSC (none) -> C527089
- J1, J10, J11, J12, J13, J14, J15, J16, J17, J18, J2, J3, J4, J5, J6, J7, J8, J9: now left out of the parts list
- SW1: Digikey (none) -> CKN10723CT-ND; LCSC (none) -> C221665; Mouser (none) -> 611-JS202011JCQN
- SW2, SW3: LCSC (none) -> C561514
Connections:
- net GND: now also JP1.2 (B); no longer D17.1 (K)
- net at U1.40 (BOOTSEL): now also TP1.1
- new net: D17.1 (K), JP1.1 (A)
- no-connect marks 10 -> 9
